File: hardware/sprint_logger.brd (EAGLE design)
At the start: 24.1 x 39.4 mm, 13 parts, among them U1 NCP1402, U2 ATMEGA168, U3 HC_05_MODIFIED

Commit message: Intial v1.6 commit
Parts:
- removed REED: M02, SparkFun-Connectors:1X02-SMD_EDGE
- added LED1: (no value), SparkFun-LED:LED-1206
- added R1: 1K, SparkFun-Passives:0805
- added R2, R3: 10K, SparkFun-Passives:0805
- added U$3: M03, petrocik:1X06-SMD_EDGE
Connections:
- net N$6 renamed SDA
- net N$7 renamed SCL
- new net KEY: R1.1, U2.25
- new net LED: R3.2, U2.23
- new net N$10: R1.2, U3.34
- new net N$6: LED1.A, R3.1
- new net STATE: U2.26, U3.32
- net GND: now also LED1.C, U$3.1; no longer REED.1
- net N$1: now also R2.1, U$3.3; no longer REED.2
- net VCC: now also R2.2, U$3.2
Routing:
- net LED: track 0.00 -> 14.7 mm, vias 0 -> 2
- net N$10: track 0.00 -> 14.5 mm
- net VCC: track 74.1 -> 85.4 mm, vias 1 -> 2
- net STATE: track 0.00 -> 11.3 mm, vias 0 -> 1
- net GND: track 47.8 -> 58.0 mm
- net KEY: track 0.00 -> 9.00 mm, vias 0 -> 1
- net N$6: track 0.00 -> 2.68 mm
- net VIN: track 18.1 -> 19.0 mm
- net N$1: track 29.7 -> 29.0 mm
Other:
- board text added: "SprintLogger v1.7"
- board text removed: "SprintLogger v1.4"
