File: hardware/sprint_logger.sch (EAGLE design)
At the start: 13 parts, among them U1 NCP1402, U2 ATMEGA168, U3 HC_05_MODIFIED

Commit message: Intial v1.6 commit
Parts:
- removed REED: M02, SparkFun-Connectors:M02
- added LED1: (no value), SparkFun-LED:LED1206
- added R1: 1K, SparkFun-Passives:RESISTOR0805-RES
- added R2, R3: 10K, SparkFun-Passives:RESISTOR0805-RES
- added U$3: M03, petrocik:M03
Connections:
- net N$6 renamed SDA
- net N$7 renamed SCL
- new net KEY: R1.1, U2.PC2(ADC2)
- new net LED: R3.2, U2.PC0(ADC0)
- new net N$10: R1.2, U3.PIO11
- new net N$6: LED1.A, R3.1
- new net STATE: U2.PC3(ADC3), U3.PIO9
- net GND: now also LED1.C, U$3.1; no longer REED.1
- net N$1: now also R2.1, U$3.3; no longer REED.2
- net VCC: now also R2.2, U$3.2
Changed lines of the file:
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@@
 <part name="GND3" library="SparkFun" deviceset="GND" device=""/>
 <part name="U$2" library="SparkFun-Connectors" deviceset="AVR_SPI_PROG3" device=""/>
-<part name="REED" library="SparkFun-Connectors" deviceset="M02" device=""/>
+<part name="U$3" library="petrocik" deviceset="M03" device=""/>
+<part name="SUPPLY1" library="SparkFun-Aesthetics" deviceset="VCC" device=""/>
+<part name="R1" library="SparkFun-Passives" deviceset="RESISTOR" device="0805-RES" value="1K"/>
+<part name="R2" library="SparkFun-Passives" deviceset="RESISTOR" device="0805-RES" value="10K"/>
+<part name="LED1" library="SparkFun-LED" deviceset="LED" device="1206"/>
+<part name="R3" library="SparkFun-Passives" deviceset="RESISTOR" device="0805-RES" value="10K"/>
+<part name="GND4" library="SparkFun-Aesthetics" deviceset="GND" device=""/>
 </parts>
 <sheets>
@@
 <instance part="R4" gate="G$1" x="106.68" y="38.1" rot="R90"/>
 <instance part="U3" gate="G$1" x="149.86" y="76.2"/>
-<instance part="GND7" gate="1" x="116.84" y="30.48" rot="R180"/>
+<instance part="GND7" gate="1" x="124.46" y="33.02" rot="R180"/>
 <instance part="U1" gate="G$1" x="104.14" y="-35.56" rot="MR0"/>
 <instance part="D3" gate="G$1" x="101.6" y="-20.32" smashed="yes">
@@
 <instance part="GND3" gate="1" x="20.32" y="-45.72"/>
 <instance part="U$2" gate="G$1" x="170.18" y="7.62"/>
-<instance part="REED" gate="G$1" x="129.54" y="25.4" rot="R180"/>
+<instance part="U$3" gate="G$1" x="139.7" y="22.86" rot="R180"/>
+<instance part="SUPPLY1" gate="1" x="114.3" y="25.4" rot="R90"/>
+<instance part="R1" gate="G$1" x="190.5" y="91.44" rot="R180"/>
+<instance part="R2" gate="G$1" x="119.38" y="20.32" rot="R90"/>
+<instance part="LED1" gate="G$1" x="106.68" y="-5.08" rot="R90"/>
+<instance part="R3" gate="G$1" x="91.44" y="-5.08" rot="R180"/>
+<instance part="GND4" gate="1" x="124.46" y="-5.08" rot="R90"/>
 </instances>
 <busses>
@@
 </segment>
 <segment>
-<pinref part="REED" gate="G$1" pin="1"/>
+<pinref part="U$3" gate="G$1" pin="1"/>
+<wire x1="132.08" y1="25.4" x2="124.46" y2="25.4" width="0.1524" layer="91"/>
+<wire x1="124.46" y1="25.4" x2="124.46" y2="30.48" width="0.1524" layer="91"/>
 <pinref part="GND7" gate="1" pin="GND"/>
-<wire x1="121.92" y1="25.4" x2="116.84" y2="25.4" width="0.1524" layer="91"/>
-<wire x1="116.84" y1="25.4" x2="116.84" y2="27.94" width="0.1524" layer="91"/>
+</segment>
+<segment>
+<pinref part="LED1" gate="G$1" pin="C"/>
+<pinref part="GND4" gate="1" pin="GND"/>
+<wire x1="111.76" y1="-5.08" x2="121.92" y2="-5.08" width="0.1524" layer="91"/>
 </segment>
 </net>
@@
 <pinref part="C2" gate="G$1" pin="+"/>
 </segment>
-</net>
-<net name="N$6" class="0">
-<segment>
-<pinref part="U2" gate="G$1" pin="PC4(ADC4/SDA)"/>
-<wire x1="83.82" y1="58.42" x2="86.36" y2="58.42" width="0.1524" layer="91"/>
-<wire x1="86.36" y1="58.42" x2="86.36" y2="83.82" width="0.1524" layer="91"/>
+<segment>
+<wire x1="114.3" y1="25.4" x2="119.38" y2="25.4" width="0.1524" layer="91"/>
+<pinref part="SUPPLY1" gate="1" pin="VCC"/>
+<pinref part="R2" gate="G$1" pin="2"/>
+<pinref part="U$3" gate="G$1" pin="2"/>
+<wire x1="132.08" y1="22.86" x2="121.92" y2="22.86" width="0.1524" layer="91"/>
+<wire x1="121.92" y1="22.86" x2="121.92" y2="25.4" width="0.1524" layer="91"/>
+<wire x1="121.92" y1="25.4" x2="119.38" y2="25.4" width="0.1524" layer="91"/>
+<junction x="119.38" y="25.4"/>
+</segment>
+</net>
+<net name="SDA" class="0">
+<segment>
 <pinref part="U$1" gate="G$1" pin="SDA"/>
 <wire x1="86.36" y1="83.82" x2="71.12" y2="83.82" width="0.1524" layer="91"/>
-</segment>
-</net>
-<net name="N$7" class="0">
-<segment>
-<pinref part="U2" gate="G$1" pin="PC5(ADC5/SCL)"/>
-<wire x1="83.82" y1="55.88" x2="88.9" y2="55.88" width="0.1524" layer="91"/>
-<wire x1="88.9" y1="55.88" x2="88.9" y2="86.36" width="0.1524" layer="91"/>
-<pinref part="U$1" gate="G$1" pin="SCL"/>
-<wire x1="88.9" y1="86.36" x2="71.12" y2="86.36" width="0.1524" layer="91"/>
-</segment>
-</net>
-<net name="N$1" class="0">
-<segment>
-<wire x1="91.44" y1="38.1" x2="91.44" y2="22.86" width="0.1524" layer="91"/>
-<pinref part="U2" gate="G$1" pin="PD3(INT1)"/>
-<wire x1="83.82" y1="38.1" x2="91.44" y2="38.1" width="0.1524" layer="91"/>
-<pinref part="REED" gate="G$1" pin="2"/>
-<wire x1="121.92" y1="22.86" x2="91.44" y2="22.86" width="0.1524" layer="91"/>
+<label x="86.36" y="83.82" size="1.27" layer="95" xref="yes"/>
+</segment>
+<segment>
+<pinref part="U2" gate="G$1" pin="PC4(ADC4/SDA)"/>
+<wire x1="83.82" y1="58.42" x2="88.9" y2="58.42" width="0.1524" layer="91"/>
+<label x="88.9" y="58.42" size="1.27" layer="95" xref="yes"/>
 </segment>
 </net>
@@
 </segment>
 </net>
+<net name="N$10" class="0">
+<segment>
+<pinref part="U3" gate="G$1" pin="PIO11"/>
+<pinref part="R1" gate="G$1" pin="2"/>
+<wire x1="175.26" y1="91.44" x2="185.42" y2="91.44" width="0.1524" layer="91"/>
+</segment>
+</net>
+<net name="N$1" class="0">
+<segment>
+<pinref part="U$3" gate="G$1" pin="3"/>
+<wire x1="132.08" y1="20.32" x2="129.54" y2="20.32" width="0.1524" layer="91"/>
+<wire x1="129.54" y1="20.32" x2="129.54" y2="15.24" width="0.1524" layer="91"/>
+<pinref part="R2" gate="G$1" pin="1"/>
+<wire x1="129.54" y1="15.24" x2="119.38" y2="15.24" width="0.1524" layer="91"/>
+<wire x1="119.38" y1="15.24" x2="101.6" y2="15.24" width="0.1524" layer="91"/>
+<wire x1="101.6" y1="15.24" x2="101.6" y2="38.1" width="0.1524" layer="91"/>
+<pinref part="U2" gate="G$1" pin="PD3(INT1)"/>
+<wire x1="101.6" y1="38.1" x2="83.82" y2="38.1" width="0.1524" layer="91"/>
+<junction x="119.38" y="15.24"/>
+</segment>
+</net>
+<net name="SCL" class="0">
+<segment>
+<pinref part="U$1" gate="G$1" pin="SCL"/>
+<wire x1="71.12" y1="86.36" x2="86.36" y2="86.36" width="0.1524" layer="91"/>
+<label x="86.36" y="86.36" size="1.27" layer="95" xref="yes"/>
+</segment>
+<segment>
+<pinref part="U2" gate="G$1" pin="PC5(ADC5/SCL)"/>
+<wire x1="83.82" y1="55.88" x2="88.9" y2="55.88" width="0.1524" layer="91"/>
+<label x="88.9" y="55.88" size="1.27" layer="95" xref="yes"/>
+</segment>
+</net>
+<net name="N$6" class="0">
+<segment>
+<pinref part="R3" gate="G$1" pin="1"/>
+<pinref part="LED1" gate="G$1" pin="A"/>
+<wire x1="96.52" y1="-5.08" x2="104.14" y2="-5.08" width="0.1524" layer="91"/>
+</segment>
+</net>
+<net name="LED" class="0">
+<segment>
+<pinref part="U2" gate="G$1" pin="PC0(ADC0)"/>
+<wire x1="83.82" y1="68.58" x2="88.9" y2="68.58" width="0.1524" layer="91"/>
+<label x="88.9" y="68.58" size="1.27" layer="95" xref="yes"/>
+</segment>
+<segment>
+<pinref part="R3" gate="G$1" pin="2"/>
+<wire x1="86.36" y1="-5.08" x2="76.2" y2="-5.08" width="0.1524" layer="91"/>
+<label x="76.2" y="-5.08" size="1.27" layer="95" rot="R180" xref="yes"/>
+</segment>
+</net>
+<net name="KEY" class="0">
+<segment>
+<pinref part="R1" gate="G$1" pin="1"/>
+<wire x1="195.58" y1="91.44" x2="203.2" y2="91.44" width="0.1524" layer="91"/>
+<label x="203.2" y="91.44" size="1.27" layer="95" xref="yes"/>
+</segment>
+<segment>
+<pinref part="U2" gate="G$1" pin="PC2(ADC2)"/>
+<wire x1="83.82" y1="63.5" x2="88.9" y2="63.5" width="0.1524" layer="91"/>
+<label x="88.9" y="63.5" size="1.27" layer="95" xref="yes"/>
+</segment>
+</net>
+<net name="STATE" class="0">
+<segment>
+<pinref part="U3" gate="G$1" pin="PIO9"/>
+<wire x1="175.26" y1="86.36" x2="182.88" y2="86.36" width="0.1524" layer="91"/>
+<label x="182.88" y="86.36" size="1.27" layer="95" xref="yes"/>
+</segment>
+<segment>
+<pinref part="U2" gate="G$1" pin="PC3(ADC3)"/>
+<wire x1="83.82" y1="60.96" x2="88.9" y2="60.96" width="0.1524" layer="91"/>
+<label x="88.9" y="60.96" size="1.27" layer="95" xref="yes"/>
+</segment>
+</net>
